Commit message: fix exercice 4

File: workshop_robot_description/urdf/ur10e_with_cube.urdf.xacro (robot description, xacro)
@@ -40,5 +40,5 @@
     <xacro:include filename="$(find ur_description)/urdf/ur_macro.xacro"/>
     <xacro:include filename="$(find workshop_robot_description)/urdf/ur.ros2_control.xacro" />
-    <xacro:arg name="ur_type" default="ur10e"/>
+    <xacro:arg name="ur_type" default="ur30"/>
     <!-- parameters for ur -->
     <xacro:arg name="tf_prefix" default="" />
@@ -83,4 +83,20 @@
         <origin xyz="0.05 0 0.06" rpy="0 0 0"/>
     </joint>
+    <link name="michel_link">
+    <visual>
+        <origin xyz="0.05 0 0.06" rpy="0 0 0"/>
+        <geometry>
+        <box size="0.5 0.03 0.04"/>
+        </geometry>
+        <material name="black">
+        <color rgba="0.05 0.05 0.05 1"/>
+        </material>
+    </visual>
+    </link>
+    <joint name="ee_to_michel" type="fixed">
+        <parent link="tool0"/>
+        <child link="michel_link"/>
+        <origin xyz="-0.2 0.5 0.00" rpy="0 0 0"/>
+    </joint>
     <xacro:ur_ros2_control
         name="ur10e"
